File: _autosave-Spore_proto.kicad_pcb (KiCad board)
At the start: 2 copper layers, 74 parts, among them J1 BATT, J2 5V IN, J3 FTDI to ESP, J4 LED OUT, J5 SENSOR, J6 SERVO, J7 MOSFET, J8 MOTOR, J9 I2C, Q1 DMG2302UK-7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

Commit message: checkpoint-pcbnew
Parts:
- added C10: 1.0uF, Capacitors_SMD:C_0805, F.Cu at (-22.0, 20.0)
- added C13: 1.0uF, Capacitors_SMD:C_0805, B.Cu at (-23.0, -13.0)
- added C14: 1.0uF, Capacitors_SMD:C_0805, F.Cu at (-13.0, 16.0)
- added C16: 1.0uF, Capacitors_SMD:C_0805, B.Cu at (23.0, -13.0)
- added D12: SK6812-RGBW, TI_led:LED_SK6812_PLCC4_5.0x5.0mm_P3.2mm, B.Cu at (-17.4, -20.7)
- added D13: SK6812-RGBW, TI_led:LED_SK6812_PLCC4_5.0x5.0mm_P3.2mm, B.Cu at (-26.6, -4.69)
- added D14: SK6812-RGBW, TI_led:LED_SK6812_PLCC4_5.0x5.0mm_P3.2mm, B.Cu at (-23.4, 13.5)
- added D15: SK6812-RGBW, TI_led:LED_SK6812_PLCC4_5.0x5.0mm_P3.2mm, B.Cu at (-9.23, 25.4)
- added D16: SK6812-RGBW, TI_led:LED_SK6812_PLCC4_5.0x5.0mm_P3.2mm, B.Cu at (9.23, 25.4)
- added D17: SK6812-RGBW, TI_led:LED_SK6812_PLCC4_5.0x5.0mm_P3.2mm, B.Cu at (23.4, 13.5)
- added D18: SK6812-RGBW, TI_led:LED_SK6812_PLCC4_5.0x5.0mm_P3.2mm, B.Cu at (26.6, -4.69)
- added D19: SK6812-RGBW, TI_led:LED_SK6812_PLCC4_5.0x5.0mm_P3.2mm, B.Cu at (17.4, -20.7)
- moved D10 333.7 mm to (-26.6, -4.69), turned to 170 degrees
- moved D11 323.9 mm to (-17.4, -20.7), turned to 130 degrees
- moved D9 288.4 mm to (-23.4, 13.5), turned to 210 degrees
- moved D5 271.1 mm to (26.6, -4.69), turned to 10 degrees
- moved D7 246.5 mm to (9.23, 25.4), turned to 290 degrees
- moved D4 217.8 mm to (17.4, -20.7), turned to 50 degrees
- moved D8 209.8 mm to (-9.23, 25.4), turned to 250 degrees
- moved D6 199.8 mm to (23.4, 13.5), turned to 330 degrees
- moved C15 163.8 mm to (-67.0, 8.09)
- moved C16 163.8 mm to (-80.2, 8.09)
- moved C17 163.8 mm to (-58.3, 8.09)
- moved C14 153.6 mm to (-47.0, -15.0)
- moved C12 150.9 mm to (-51.0, -1.00)
- moved C11 146.3 mm to (-23.0, -13.0), turned to 144 degrees
- moved C13 140.4 mm to (-50.0, -7.00)
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Other:
- board outline added: 84.5 x 80.3 mm
