File: Spore_proto.sch (KiCad schematic (older format))
At the start: 73 parts

Commit message: aesthetic adjustments + footprint assignment
Parts:
- J2: renamed from J?; footprint Connectors_JST:JST_PH_B2B-PH-K_02x2.00mm_Straight -> Connectors_JST:JST_EH_B02B-EH-A_02x2.50mm_Straight
- J4, J5, J6, J7: renamed from J?; footprint (none) -> Connectors_JST:JST_EH_B03B-EH-A_03x2.50mm_Straight
- J8, J9: renamed from J?; footprint (none) -> Connectors_JST:JST_EH_B04B-EH-A_04x2.50mm_Straight
- gave numbers to parts that had none: 66

Commit message: added power switch (allows charging while off), minor tweaks, footprint assignments
Parts:
- added SW?: PWR, symbol SW_DPST
- D1: footprint (none) -> Diodes_SMD:D_SOD-123F
- JP3: symbol Jumper_NO_Small -> Jumper_NC_Small
- JP4: value BATT_EN -> BATT_SENSE
- R15: value 100 -> 330
Connections:
- net +BATT: now also SW?.5; no longer C10.1, C11.1, C12.1, C13.1, C14.1, C15.1, C16.1, C17.1, C8.1, C9.1, D10.3 (VDD), D11.3 (VDD), D12.3 (VDD), D13.3 (VDD), D14.3 (VDD), D15.3 (VDD), D16.3 (VDD), D17.3 (VDD), D18.3 (VDD), D19.3 (VDD), D4.3 (VDD), D5.3 (VDD), D6.3 (VDD), D7.3 (VDD), D8.3 (VDD), D9.3 (VDD), J4.2 (P2)
- net V_IN: now also SW?.3; no longer D1.1 (K), JP3.2
- new net: D1.1 (K), JP3.2, SW?.2
- new net V_BATT: C10.1, C11.1, C12.1, C13.1, C14.1, C15.1, C16.1, C17.1, C8.1, C9.1, D10.3 (VDD), D11.3 (VDD), D12.3 (VDD), D13.3 (VDD), D14.3 (VDD), D15.3 (VDD), D16.3 (VDD), D17.3 (VDD), D18.3 (VDD), D19.3 (VDD), D4.3 (VDD), D5.3 (VDD), D6.3 (VDD), D7.3 (VDD), D8.3 (VDD), D9.3 (VDD), J4.2 (P2), SW?.6
Other:
- note added: "STYLE\nTBD"
- note removed: "TBD"
- moved on the sheet: C1, C2, C3, D1, D2, D3, R3, R4, R5, R6, U1, U2

Commit message: few tweaks. Pre-PCBNew
Parts:
- JP1, JP2, JP3, JP4: footprint (none) -> TI_conn:JMP
- R3: value 2.2k -> 4.7k
- SW1: renamed from SW?; value PWR -> JS202011AQN; footprint (none) -> TI_switches:SW_Micro_DPDT
- renumbered SW1 to SW2, SW2 to SW3
Connections:
- net LED_IN is gone; now on net TX: R15.2
Other:
- note added: "(this is the \nDMA pin)"
Changed lines of the file:
@@
 Title "SPORE PCB"
 Date "2018-03-06"
-Rev "0.0.1"
+Rev "0.0.2"
 Comp ""
 Comment1 "SPORE"
@@
 BOOTLOAD
 $Comp
-L SW_Push SW2
+L SW_Push SW3
 U 1 1 5A9F3863
 P 1450 4100
-F 0 "SW2" H 1500 4200 50  0000 L CNN
+F 0 "SW3" H 1500 4200 50  0000 L CNN
 F 1 "Reset" H 1450 4040 50  0000 C CNN
 F 2 "Buttons_Switches_SMD:SW_SPST_PTS645" H 1450 4300 50  0001 C CNN
@@
 $EndComp
 $Comp
-L SW_Push SW1
+L SW_Push SW2
 U 1 1 5A9F38AC
 P 1450 3100
-F 0 "SW1" H 1500 3200 50  0000 L CNN
+F 0 "SW2" H 1500 3200 50  0000 L CNN
 F 1 "Bootload" H 1450 3040 50  0000 C CNN
 F 2 "Buttons_Switches_SMD:SW_SPST_PTS645" H 1450 3300 50  0001 C CNN
@@
 P 1000 1300
 F 0 "R3" V 900 1250 50  0000 L TNN
-F 1 "2.2k" V 1050 1250 50  0000 L TNN
+F 1 "4.7k" V 1050 1250 50  0000 L TNN
 F 2 "Resistors_SMD:R_0805" H 1000 1300 50  0001 C CNN
 F 3 "" H 1000 1300 50  0001 C CNN
@@
 F 0 "JP3" H 2900 1000 50  0000 C CNN
 F 1 "EXT_EN" H 3150 1000 50  0000 C CNN
-F 2 "" H 3050 1100 50  0001 C CNN
+F 2 "TI_conn:JMP" H 3050 1100 50  0001 C CNN
 F 3 "" H 3050 1100 50  0001 C CNN
 	1    3050 1100
@@
 	1    0    0    -1
 $EndComp
-Text Label 750  5400 0    60   ~ 0
-LED_IN
+Text Label 900  5400 0    60   ~ 0
+TX
 Text Notes 2250 2250 0    60   ~ 0
 Connectors
@@
 F 0 "JP1" V 8150 1050 50  0000 L CNN
 F 1 "3v3_EN" V 8250 1050 50  0000 L CNN
-F 2 "" H 8200 1000 50  0001 C CNN
+F 2 "TI_conn:JMP" H 8200 1000 50  0001 C CNN
 F 3 "" H 8200 1000 50  0001 C CNN
 	1    8200 1000
@@
 F 0 "JP2" V 8550 1050 50  0000 L CNN
 F 1 "EXT_EN" V 8650 1050 50  0000 L CNN
-F 2 "" H 8600 1000 50  0001 C CNN
+F 2 "TI_conn:JMP" H 8600 1000 50  0001 C CNN
 F 3 "" H 8600 1000 50  0001 C CNN
 	1    8600 1000
@@
 F 0 "JP4" V 9600 5400 50  0000 L CNN
 F 1 "BATT_SENSE" V 9700 5400 50  0000 L CNN
-F 2 "" H 9650 5350 50  0001 C CNN
+F 2 "TI_conn:JMP" H 9650 5350 50  0001 C CNN
 F 3 "" H 9650 5350 50  0001 C CNN
 	1    9650 5350
@@
 $EndComp
 $Comp
-L GND #PWR044
+L GND #PWR042
 U 1 1 5AA2A5C1
 P 2800 4200
-F 0 "#PWR044" H 2800 3950 50  0001 C CNN
+F 0 "#PWR042" H 2800 3950 50  0001 C CNN
 F 1 "GND" H 2800 4050 50  0000 C CNN
 F 2 "" H 2800 4200 50  0001 C CNN
@@
 $EndComp
 $Comp
-L +3.3V #PWR045
+L +3.3V #PWR043
 U 1 1 5AA2A831
 P 2800 3800
-F 0 "#PWR045" H 2800 3650 50  0001 C CNN
+F 0 "#PWR043" H 2800 3650 50  0001 C CNN
 F 1 "+3.3V" H 2800 3940 50  0000 C CNN
 F 2 "" H 2800 3800 50  0001 C CNN
@@
 $EndComp
 $Comp
-L GND #PWR046
+L GND #PWR044
 U 1 1 5AA2B823
 P 3700 4200
-F 0 "#PWR046" H 3700 3950 50  0001 C CNN
+F 0 "#PWR044" H 3700 3950 50  0001 C CNN
 F 1 "GND" H 3700 4050 50  0000 C CNN
 F 2 "" H 3700 4200 50  0001 C CNN
@@
 $EndComp
 $Comp
-L +3.3V #PWR047
+L +3.3V #PWR045
 U 1 1 5AA2D3AC
 P 9000 4950
-F 0 "#PWR047" H 9000 4800 50  0001 C CNN
+F 0 "#PWR045" H 9000 4800 50  0001 C CNN
 F 1 "+3.3V" H 9000 5090 50  0000 C CNN
 F 2 "" H 9000 4950 50  0001 C CNN
@@
 $EndComp
 $Comp
-L GND #PWR048
+L GND #PWR046
 U 1 1 5AA2DAAB
 P 8900 5500
-F 0 "#PWR048" H 8900 5250 50  0001 C CNN
+F 0 "#PWR046" H 8900 5250 50  0001 C CNN
 F 1 "GND" H 8900 5350 50  0000 C CNN
 F 2 "" H 8900 5500 50  0001 C CNN
@@
 $EndComp
 $Comp
-L +3.3V #PWR049
+L +3.3V #PWR047
 U 1 1 5AA30915
 P 10350 2650
-F 0 "#PWR049" H 10350 2500 50  0001 C CNN
+F 0 "#PWR047" H 10350 2500 50  0001 C CNN
 F 1 "+3.3V" H 10350 2790 50  0000 C CNN
 F 2 "" H 10350 2650 50  0001 C CNN
@@
 $EndComp
 $Comp
-L GND #PWR050
+L GND #PWR048
 U 1 1 5AA3CD30
 P 4550 4200
-F 0 "#PWR050" H 4550 3950 50  0001 C CNN
+F 0 "#PWR048" H 4550 3950 50  0001 C CNN
 F 1 "GND" H 4550 4050 50  0000 C CNN
 F 2 "" H 4550 4200 50  0001 C CNN
@@
 V_IN
 $Comp
-L +5V #PWR051
+L +5V #PWR049
 U 1 1 5AA3EEB8
 P 4800 2650
-F 0 "#PWR051" H 4800 2500 50  0001 C CNN
+F 0 "#PWR049" H 4800 2500 50  0001 C CNN
 F 1 "+5V" H 4800 2790 50  0000 C CNN
 F 2 "" H 4800 2650 50  0001 C CNN
@@
 $EndComp
 $Comp
-L GND #PWR052
+L GND #PWR050
 U 1 1 5AA5712D
 P 5500 3100
-F 0 "#PWR052" H 5500 2850 50  0001 C CNN
+F 0 "#PWR050" H 5500 2850 50  0001 C CNN
 F 1 "GND" H 5500 2950 50  0000 C CNN
 F 2 "" H 5500 3100 50  0001 C CNN
@@
 STYLE\nTBD
 $Comp
-L SW_DPST SW?
+L SW_DPST SW1
 U 1 1 5AA9F468
 P 3650 1000
-F 0 "SW?" H 3500 1200 50  0000 C CNN
-F 1 "PWR" H 3650 800 50  0000 C CNN
-F 2 "" H 3650 1000 50  0001 C CNN
+F 0 "SW1" H 3500 1200 50  0000 C CNN
+F 1 "JS202011AQN" H 3650 800 50  0000 C CNN
+F 2 "TI_switches:SW_Micro_DPDT" H 3650 1000 50  0001 C CNN
 F 3 "" H 3650 1000 50  0001 C CNN
 	1    3650 1000
@@
 	1300 5400 1350 5400
 Wire Wire Line
-	750  5400 1100 5400
+	900  5400 1100 5400
 Connection ~ 1850 7100
 Connection ~ 1850 7400
@@
 Wire Wire Line
 	3300 900  3450 900
+Text Notes 750  5750 0    60   ~ 0
+(this is the \nDMA pin)
 $EndSCHEMATC

Commit message: checkpoint-pcbnew
Parts:
- J3: footprint Pin_Headers:Pin_Header_Straight_1x06_Pitch2.54mm_SMD_Pin1Right -> Pin_Headers:Pin_Header_Straight_1x06_Pitch2.54mm
Changed lines of the file:
@@
 F 0 "J3" H 4300 2550 50  0000 C CNN
 F 1 "FTDI to ESP" V 4400 2900 50  0000 C CNN
-F 2 "Pin_Headers:Pin_Header_Straight_1x06_Pitch2.54mm_SMD_Pin1Right" H 4300 2900 50  0001 C CNN
+F 2 "Pin_Headers:Pin_Header_Straight_1x06_Pitch2.54mm" H 4300 2900 50  0001 C CNN
 F 3 "" H 4300 2900 50  0001 C CNN
 	1    4300 2900

Commit message: complex pcb layout + some footprint changes
Parts:
- added C18: 0.1uF, Capacitors_SMD:C_0805, symbol C_Small
- JP1: footprint TI_conn:JMP -> TI_conn:JMP_NO
- R1, R10, R11, R12, R13, R14, R15, R16, R17, R2, R3, R4, R5, R6, R7, R8, R9: footprint Resistors_SMD:R_0805 -> Capacitors_SMD:C_0805
Connections:
- net +5V: now also D2.2 (A), C18.1
- net GND: now also C18.2; no longer D2.1 (K)
- net at R3.2: now also D2.1 (K); no longer D2.2 (A)
Other:
- moved on the sheet: C1, C2, C3, D1, D2, D3, JP3, R3, R4, R5, R6, SW1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
