File: Spore_proto.kicad_pcb (KiCad board)
At the start: 2 copper layers, 74 parts, among them J1 BATT, J2 5V IN, J3 FTDI to ESP, J4 LED OUT, J5 SENSOR, J6 SERVO, J7 MOSFET, J8 MOTOR, J9 I2C, Q1 DMG2302UK-7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

Commit message: checkpoint-pcbnew
Parts:
- moved D13 129.6 mm to (149.0, 155.2)
- moved U4 97.7 mm to (46.9, 45.0)
- moved D5 97.3 mm to (149.6, 147.0)
- moved D14 80.2 mm to (157.5, 155.2)
- moved D10 76.6 mm to (190.8, 147.2)
- moved D12 61.2 mm to (140.6, 155.3)
- moved D11 57.0 mm to (199.0, 147.2)
- moved D7 54.3 mm to (165.9, 147.1)
- moved D9 46.8 mm to (182.4, 147.1)
- moved D15 27.3 mm to (166.1, 155.4)
- moved D16 18.8 mm to (174.0, 155.4)
- moved D8 18.4 mm to (174.1, 147.2)
- moved D19 11.8 mm to (199.1, 155.5)
- moved D6 10.6 mm to (157.6, 146.9)
- moved D4 9.79 mm to (140.7, 146.9)
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Other:
- board outline added: 84.5 x 80.3 mm
- net class Default: trace_width 0.25 -> 0.2
- net class PWR added: clearance 0.2, trace_width 0.2, via_dia 0.6, via_drill 0.4
- rule trace_min: 0.2 -> 0.16
- rule via_min_drill: 0.3 -> 0.25
- rule via_min_size: 0.4 -> 0.51
Changed lines of the file:
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@@
     (links 172)
     (no_connects 172)
-    (area 0 0 0 0)
+    (area 20.715572 35.539 284.319429 159.075)
     (thickness 1.6)
-    (drawings 0)
+    (drawings 10)
     (tracks 0)
     (zones 0)
@@
     (0 F.Cu signal)
     (31 B.Cu signal)
-    (32 B.Adhes user)
-    (33 F.Adhes user)
     (34 B.Paste user)
     (35 F.Paste user)
@@
     (38 B.Mask user)
     (39 F.Mask user)
-    (40 Dwgs.User user)
     (41 Cmts.User user)
-    (42 Eco1.User user)
-    (43 Eco2.User user)
     (44 Edge.Cuts user)
     (45 Margin user)
     (46 B.CrtYd user)
     (47 F.CrtYd user)
-    (48 B.Fab user)
-    (49 F.Fab user)
   )
   (setup
-    (last_trace_width 0.25)
+    (last_trace_width 0.2)
     (trace_clearance 0.2)
     (zone_clearance 0.508)
     (zone_45_only no)
-    (trace_min 0.2)
+    (trace_min 0.16)
     (segment_width 0.2)
     (edge_width 0.15)
     (via_size 0.6)
     (via_drill 0.4)
-    (via_min_size 0.4)
-    (via_min_drill 0.3)
-    (uvia_size 0.3)
-    (uvia_drill 0.1)
+    (via_min_size 0.51)
+    (via_min_drill 0.25)
+    (uvia_size 0.6)
+    (uvia_drill 0.4)
     (uvias_allowed no)
-    (uvia_min_size 0.2)
-    (uvia_min_drill 0.1)
+    (uvia_min_size 0)
+    (uvia_min_drill 0)
     (pcb_text_width 0.3)
     (pcb_text_size 1.5 1.5)
@@
     (pad_to_mask_clearance 0.2)
     (aux_axis_origin 0 0)
-    (visible_elements FFFFE77F)
+    (visible_elements FFFFEF7F)
     (pcbplotparams
       (layerselection 0x00030_80000001)
@@
   (net_class Default "This is the default net class."
     (clearance 0.2)
-    (trace_width 0.25)
+    (trace_width 0.2)
     (via_dia 0.6)
     (via_drill 0.4)
-    (uvia_dia 0.3)
-    (uvia_drill 0.1)
-    (add_net +3V3)
-    (add_net +5V)
-    (add_net +BATT)
+    (uvia_dia 0.6)
+    (uvia_drill 0.4)
     (add_net /A0)
     (add_net /BOOTLOAD)
@@
     (add_net /EN)
     (add_net /LED_OUT)
-    (add_net /MOS_OUT)
-    (add_net /M_OUT1)
-    (add_net /M_OUT2)
     (add_net /RST)
     (add_net /RX)
@@
     (add_net /SERVO)
     (add_net /TX)
-    (add_net /V_BATT)
-    (add_net /V_IN)
-    (add_net GND)
     (add_net "Net-(C4-Pad1)")
     (add_net "Net-(D1-Pad1)")
@@
     (add_net "Net-(U2-Pad4)")
   )
+  (net_class PWR ""
+    (clearance 0.2)
+    (trace_width 0.2)
+    (via_dia 0.6)
+    (via_drill 0.4)
+    (uvia_dia 0.6)
+    (uvia_drill 0.4)
+    (add_net +3V3)
+    (add_net +5V)
+    (add_net +BATT)
+    (add_net /MOS_OUT)
+    (add_net /M_OUT1)
+    (add_net /M_OUT2)
+    (add_net /V_BATT)
+    (add_net /V_IN)
+    (add_net GND)
+  )
   (module Capacitors_SMD:C_0805 (layer F.Cu)
     (at 23.352 109.22)
@@
   )
   (module TI_led:LED_SK6812_PLCC4_5.0x5.0mm_P3.2mm (layer F.Cu)
-    (at 147.828145 153.67)
+    (at 140.716 146.939)
     (descr https://cdn-shop.adafruit.com/product-files/1138/SK6812+LED+datasheet+.pdf)
     (tags "LED RGB NeoPixel")
@@
   )
   (module TI_led:LED_SK6812_PLCC4_5.0x5.0mm_P3.2mm (layer F.Cu)
-    (at 246.665752 153.67)
+    (at 149.643 146.99)
     (descr https://cdn-shop.adafruit.com/product-files/1138/SK6812+LED+datasheet+.pdf)
     (tags "LED RGB NeoPixel")
@@
   )
   (module TI_led:LED_SK6812_PLCC4_5.0x5.0mm_P3.2mm (layer F.Cu)
-    (at 165.798619 153.67)
+    (at 157.607 146.939)
     (descr https://cdn-shop.adafruit.com/product-files/1138/SK6812+LED+datasheet+.pdf)
     (tags "LED RGB NeoPixel")
@@
   )
   (module TI_led:LED_SK6812_PLCC4_5.0x5.0mm_P3.2mm (layer F.Cu)
-    (at 219.710041 153.67)
+    (at 165.862 147.066)
     (descr https://cdn-shop.adafruit.com/product-files/1138/SK6812+LED+datasheet+.pdf)
     (tags "LED RGB NeoPixel")
@@
   )
   (module TI_led:LED_SK6812_PLCC4_5.0x5.0mm_P3.2mm (layer F.Cu)
-    (at 156.813382 153.67)
+    (at 174.08 147.244)
     (descr https://cdn-shop.adafruit.com/product-files/1138/SK6812+LED+datasheet+.pdf)
     (tags "LED RGB NeoPixel")
@@
   )
   (module TI_led:LED_SK6812_PLCC4_5.0x5.0mm_P3.2mm (layer F.Cu)
-    (at 228.695278 153.67)
+    (at 182.372 147.066)
     (descr https://cdn-shop.adafruit.com/product-files/1138/SK6812+LED+datasheet+.pdf)
     (tags "LED RGB NeoPixel")
@@
   )
   (module TI_led:LED_SK6812_PLCC4_5.0x5.0mm_P3.2mm (layer F.Cu)
-    (at 267.118 153.746)
+    (at 190.754 147.193)
     (descr https://cdn-shop.adafruit.com/product-files/1138/SK6812+LED+datasheet+.pdf)
     (tags "LED RGB NeoPixel")
@@
   )
   (module TI_led:LED_SK6812_PLCC4_5.0x5.0mm_P3.2mm (layer F.Cu)
-    (at 255.650989 153.67)
+    (at 199.009 147.193)
     (descr https://cdn-shop.adafruit.com/product-files/1138/SK6812+LED+datasheet+.pdf)
     (tags "LED RGB NeoPixel")
@@
   )
   (module TI_led:LED_SK6812_PLCC4_5.0x5.0mm_P3.2mm (layer F.Cu)
-    (at 201.739567 153.67)
+    (at 140.589 155.321)
     (descr https://cdn-shop.adafruit.com/product-files/1138/SK6812+LED+datasheet+.pdf)
     (tags "LED RGB NeoPixel")
@@
   )
   (module TI_led:LED_SK6812_PLCC4_5.0x5.0mm_P3.2mm (layer F.Cu)
-    (at 278.548 154)
+    (at 148.971 155.194)
     (descr https://cdn-shop.adafruit.com/product-files/1138/SK6812+LED+datasheet+.pdf)
     (tags "LED RGB NeoPixel")
@@
   )
   (module TI_led:LED_SK6812_PLCC4_5.0x5.0mm_P3.2mm (layer F.Cu)
-    (at 237.680515 153.67)
+    (at 157.517 155.245)
     (descr https://cdn-shop.adafruit.com/product-files/1138/SK6812+LED+datasheet+.pdf)
     (tags "LED RGB NeoPixel")
@@
   )
   (module TI_led:LED_SK6812_PLCC4_5.0x5.0mm_P3.2mm (layer F.Cu)
-    (at 138.842908 153.67)
+    (at 166.079 155.397)
     (descr https://cdn-shop.adafruit.com/product-files/1138/SK6812+LED+datasheet+.pdf)
     (tags "LED RGB NeoPixel")
@@
   )
   (module TI_led:LED_SK6812_PLCC4_5.0x5.0mm_P3.2mm (layer F.Cu)
-    (at 192.75433 153.67)
+    (at 173.99 155.448)
     (descr https://cdn-shop.adafruit.com/product-files/1138/SK6812+LED+datasheet+.pdf)
     (tags "LED RGB NeoPixel")
@@
   )
   (module TI_led:LED_SK6812_PLCC4_5.0x5.0mm_P3.2mm (layer F.Cu)
-    (at 174.783856 153.67)
+    (at 182.372 155.448)
     (descr https://cdn-shop.adafruit.com/product-files/1138/SK6812+LED+datasheet+.pdf)
     (tags "LED RGB NeoPixel")
@@
   )
   (module TI_led:LED_SK6812_PLCC4_5.0x5.0mm_P3.2mm (layer F.Cu)
-    (at 183.769093 153.67)
+    (at 190.59 155.499)
     (descr https://cdn-shop.adafruit.com/product-files/1138/SK6812+LED+datasheet+.pdf)
     (tags "LED RGB NeoPixel")
@@
   )
   (module TI_led:LED_SK6812_PLCC4_5.0x5.0mm_P3.2mm (layer F.Cu)
-    (at 210.724804 153.67)
+    (at 199.099 155.499)
     (descr https://cdn-shop.adafruit.com/product-files/1138/SK6812+LED+datasheet+.pdf)
     (tags "LED RGB NeoPixel")
@@
   )
   (module ESP8266:ESP-12E_Brendan (layer F.Cu)
-    (at 140.828 71.661)
+    (at 46.863 44.958)
     (descr "Module, ESP-8266, ESP-12, 16 pad, SMD")
     (tags "Module ESP-8266 ESP8266")
@@
     )
   )
+  (gr_line (start -111.719119 60.196953) (end -103.464109 34.790644) (layer Edge.Cuts) (width 0.1))
+  (gr_line (start -82.847774 19.812) (end -56.134 19.812) (layer Edge.Cuts) (width 0.1))
+  (gr_line (start -35.137394 84.432908) (end -56.749291 100.13487) (layer Edge.Cuts) (width 0.1))
+  (gr_line (start -103.464109 34.790644) (end -82.847774 19.812) (layer Edge.Cuts) (width 0.1))
+  (gr_line (start -35.517665 34.790644) (end -27.262655 60.196953) (layer Edge.Cuts) (width 0.1))
+  (gr_line (start -27.262655 60.196953) (end -35.137394 84.432908) (layer Edge.Cuts) (width 0.1))
+  (gr_line (start -56.749291 100.13487) (end -82.232483 100.13487) (layer Edge.Cuts) (width 0.1))
+  (gr_line (start -82.232483 100.13487) (end -103.84438 84.432908) (layer Edge.Cuts) (width 0.1))
+  (gr_line (start -103.84438 84.432908) (end -111.719119 60.196953) (layer Edge.Cuts) (width 0.1))
+  (gr_line (start -56.134 19.812) (end -35.517665 34.790644) (layer Edge.Cuts) (width 0.1))
 )

Commit message: basic pcb layout done
Parts:
- C12, C13, C14, C15, C16, D12, D13, D14, D15, D16, D17, D18, D19: moved to B.Cu
- J3: footprint Pin_Headers:Pin_Header_Straight_1x06_Pitch2.54mm -> TI_conn:Pin_Header_Straight_1x06_Pitch2.54mm
- moved J6 307.2 mm to (-35.8, -9.12), turned to 72 degrees
- moved J5 287.9 mm to (-23.5, -28.5), turned to 36 degrees
- moved D11 273.9 mm to (-17.4, -20.7), turned to 130 degrees
- moved J9 271.4 mm to (-34.2, 13.4), turned to 108 degrees
- moved D10 265.2 mm to (-26.6, -4.69), turned to 170 degrees
- moved D19 253.1 mm to (17.4, -20.7), turned to 230 degrees
- moved SW1 247.7 mm to (5.50, 36.0)
- moved D9 245.3 mm to (-23.4, 13.5), turned to 210 degrees
- moved J1 239.8 mm to (-1.00, -7.00)
- moved D13 237.5 mm to (-26.6, -4.69), turned to 350 degrees
- moved D12 236.5 mm to (-17.4, -20.7), turned to 310 degrees
- moved D14 229.8 mm to (-23.4, 13.5), turned to 30 degrees
- moved J2 229.6 mm to (-7.00, 36.0)
- moved D18 229.3 mm to (26.6, -4.69), turned to 190 degrees
- moved J4 224.1 mm to (19.5, -31.0), turned to 324 degrees
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
Commit message: complex pcb layout + some footprint changes
Parts:
- added C18: 0.1uF, Capacitors_SMD:C_0805, F.Cu at (16.5, 10.0)
- C17: moved to B.Cu
- C4, C5: footprint Capacitors_SMD:C_0805 -> Capacitors_SMD:C_0603
- J3: footprint TI_conn:Pin_Header_Straight_1x06_Pitch2.54mm -> Pin_Headers:Pin_Header_Straight_1x06_Pitch2.54mm
- JP1: footprint TI_conn:JMP -> TI_conn:JMP_NO
- R1: footprint Resistors_SMD:R_0805 -> Capacitors_SMD:C_0603
- R10, R11, R12, R13, R14, R15, R16, R17, R2, R3, R4, R5, R6, R7, R8, R9: footprint Resistors_SMD:R_0805 -> Capacitors_SMD:C_0805
- moved R1 149.4 mm to (-25.5, 4.50)
- moved JP2 138.7 mm to (-36.8, 0.47), turned to 288 degrees
- moved JP1 136.1 mm to (-38.8, 1.12), turned to 288 degrees
- moved R7 129.7 mm to (-14.0, -7.50), turned to 270 degrees
- moved R14 129.0 mm to (-13.5, 8.50)
- moved C1 127.7 mm to (16.9, -7.81), turned to 90 degrees
- moved R16 126.1 mm to (-9.50, 6.50), turned to 180 degrees
- moved R4 123.4 mm to (0.00, 32.0), turned to 180 degrees
- moved R17 122.5 mm to (-9.50, 8.50), turned to 180 degrees
- moved C3 119.3 mm to (6.50, 10.0), turned to 90 degrees
- moved C2 117.6 mm to (6.94, -7.81), turned to 90 degrees
- moved U3 114.9 mm to (-28.5, 6.00)
- moved R9 112.4 mm to (-11.0, -27.0)
- moved JP3 110.2 mm to (-4.00, 32.0)
- moved R13 105.1 mm to (-11.0, -24.5)
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Connections:
- D2 pad 1: GND -> Net-(D2-Pad1)
- D2 pad 2: Net-(D2-Pad2) -> +5V
- R3 pad 2: Net-(D2-Pad2) -> Net-(D2-Pad1)
- SW1 pad 1: Net-(D1-Pad1) -> (no net)
- SW1 pad 2: /V_IN -> Net-(D1-Pad1)
- SW1 pad 3: +BATT -> /V_IN
- SW1 pad 4: /V_BATT -> (no net)
- SW1 pad 5: (no net) -> +BATT
- SW1 pad 6: (no net) -> /V_BATT

Commit message: gerbers, BOM, etc for PCB fab
Parts:
- added G***: LOGO, TI_logo:SPORE_logo_27mm_FSilk, B.Cu at (100.3, 88.5)
- added G***: LOGO, TI_logo:TI_logo_9.5mm_FSilk, F.Cu at (87.9, 110.0)
- added REF***: OSHW-Logo_7.5x8mm_SilkScreen, Symbols:OSHW-Logo_7.5x8mm_SilkScreen, B.Cu at (99.8, 127.3)
- U3: footprint Housings_DFN_QFN:DFN-8-1EP_2x2mm_Pitch0.5mm -> TI_ic:DFN-8-1EP_2x2mm_Pitch0.5mm
- moved R12 142.5 mm to (111.0, 82.0)
- moved D3 141.8 mm to (99.5, 136.5)
- moved C10 141.4 mm to (83.0, 120.0)
- moved C11 141.4 mm to (77.0, 87.0)
- moved C12 141.4 mm to (86.0, 76.5), turned to 130 degrees
- moved C13 141.4 mm to (77.0, 87.0), turned to 144 degrees
- moved C14 141.4 mm to (83.0, 120.0), turned to 234 degrees
- moved C15 141.4 mm to (117.0, 120.0), turned to 306 degrees
- moved C16 141.4 mm to (123.0, 87.0), turned to 36 degrees
- moved C17 141.4 mm to (114.0, 76.5), turned to 50 degrees
- moved C4 141.4 mm to (70.0, 103.0)
- moved C5 141.4 mm to (73.0, 103.0)
- moved C6 141.4 mm to (89.0, 85.5)
- moved C7 141.4 mm to (89.0, 83.0)
- moved C8 141.4 mm to (123.0, 87.0)
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Connections:
- J1 pad 1: GND -> +BATT
- J1 pad 2: +BATT -> GND
- U3 pad 9: (no net) -> GND
Routing:
- net GND: track 0.00 -> 951.1 mm, vias 0 -> 132
- net /V_BATT: track 0.00 -> 318.7 mm, vias 0 -> 2
- net +3V3: track 0.00 -> 209.3 mm, vias 0 -> 17
- net /V_IN: track 0.00 -> 195.5 mm, vias 0 -> 10
- net +BATT: track 0.00 -> 132.7 mm, vias 0 -> 10
- net /RST: track 0.00 -> 93.2 mm, vias 0 -> 4
- net /BOOTLOAD: track 0.00 -> 83.8 mm, vias 0 -> 2
- net /TX: track 0.00 -> 80.4 mm
- net /RX: track 0.00 -> 76.0 mm
- net +5V: track 0.00 -> 71.8 mm, vias 0 -> 7
- net /SDA: track 0.00 -> 55.7 mm
- net /SCL: track 0.00 -> 53.2 mm
- net /CTL_DRV1: track 0.00 -> 41.2 mm, vias 0 -> 2
- net /CTL_DRV2: track 0.00 -> 40.8 mm, vias 0 -> 2
- net /SERVO: track 0.00 -> 31.6 mm, vias 0 -> 2
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- added copper zone on B.Cu, net +3V3
- added copper zone on F.Cu, net +3V3
- added copper zone on B.Cu, net +5V
- added copper zone on F.Cu, net +5V
- added copper zone on B.Cu, net +BATT
- added copper zone on F.Cu, net +BATT
- added copper zone on B.Cu, net /V_IN
- added copper zone on F.Cu, net /V_IN
- added copper zone on B.Cu, net GND
- added copper zone on F.Cu, net GND
- added copper zone on F.Cu, net Net-(C4-Pad1)
Other:
- outline, holes or cut-outs redrawn
- net class BIG_PWR added: clearance 0.25, trace_width 0.4, via_dia 0.6, via_drill 0.4
- net class PWR: clearance 0.2 -> 0.25; trace_width 0.2 -> 0.3
- board text added: "*!"
- board text added: "+ BATT -"
- board text added: "+5V"
- board text added: "-CHRG"
- board text added: "-LED 0"
- board text added: "-LED 8"
- board text added: "3v3 SDA GND SCL"
- board text added: "<-"
- board text added: "BAT_SNS"
- board text added: "BBM"
- board text added: "BLK"
- board text added: "BOOTLOAD"
- board text added: "DATA VIN GND"
- board text added: "FTDI"
- board text added: "GND VIN OUT"
- board text added: "GND nc +5 TX RX nc"
- board text added: "GRN"
- board text added: "I"
- board text added: "I2C"
- board text added: "IN 3v3 GND"
- board text added: "LED OUT"
- board text added: "M1 M2 VIN VIN"
- board text added: "MOSFET"
- board text added: "MOTOR"
- board text added: "O"
- board text added: "OUT V_BATT GND"
- board text added: "RESET"
- board text added: "SENSOR"
- board text added: "SERVO"
- board text added: "SPORE v0.0.3"
