File: SPORE_EDA/kicad_project/Spore.sch (KiCad schematic (older format))
At the start: 75 parts, among them J1 BATT, J2 5V IN, J3 FTDI to ESP, J4 LED OUT, J5 SENSOR, J6 SERVO, J7 MOSFET, J8 MOTOR, J9 I2C, Q1 DMG2302UK-7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

Commit message: some PCB schematic revisions for final hardware
Parts:
- D1: footprint Diodes_SMD:D_SOD-123F -> TI_ic:SOD-123F
- R14: value 100k -> 220k
Connections:
- net +BATT: no longer R14.1
- net V_BATT: now also R14.1
Other:
- note removed: "- Prob. just 10-22uF bulk cap. instead \n of 100uF"
- moved on the sheet: C6, C7, R10, R11, R12, R9, U4

Commit message: updated schematic in prep for next H/W version
Parts:
- JP3: footprint TI_conn:JMP -> TI_conn:JMP_NO; symbol Jumper_NC_Small -> Jumper_NO_Small
Connections:
- net SENSOR: now also JP4.1, R14.2
- net V_IN: now also C4.1, JP1.2, JP2.2, U3.1 (VM)
Changed lines of the file:
@@
 $EndComp
 $Comp
-L +BATT #PWR024
+L +BATT #PWR023
 U 1 1 5A9FC41A
 P 2850 2650
-F 0 "#PWR024" H 2850 2500 50  0001 C CNN
+F 0 "#PWR023" H 2850 2500 50  0001 C CNN
 F 1 "+BATT" H 2850 2790 50  0000 C CNN
 F 2 "" H 2850 2650 50  0001 C CNN
@@
 $EndComp
 $Comp
-L +5V #PWR025
+L +5V #PWR024
 U 1 1 5A9FC9CB
 P 2950 800
-F 0 "#PWR025" H 2950 650 50  0001 C CNN
+F 0 "#PWR024" H 2950 650 50  0001 C CNN
 F 1 "+5V" H 2950 940 50  0000 C CNN
 F 2 "" H 2950 800 50  0001 C CNN
@@
 $EndComp
 $Comp
-L +5V #PWR026
+L +5V #PWR025
 U 1 1 5A9FEDAE
 P 1000 800
-F 0 "#PWR026" H 1000 650 50  0001 C CNN
+F 0 "#PWR025" H 1000 650 50  0001 C CNN
 F 1 "+5V" H 1000 940 50  0000 C CNN
 F 2 "" H 1000 800 50  0001 C CNN
@@
 - ALT charge: MCP73833/4 (1.1A max)
 $Comp
-L +BATT #PWR027
+L +BATT #PWR026
 U 1 1 5AA00E70
 P 2600 800
-F 0 "#PWR027" H 2600 650 50  0001 C CNN
+F 0 "#PWR026" H 2600 650 50  0001 C CNN
 F 1 "+BATT" H 2600 940 50  0000 C CNN
 F 2 "" H 2600 800 50  0001 C CNN
@@
 $EndComp
 $Comp
-L GND #PWR028
+L GND #PWR027
 U 1 1 5AA01571
 P 2200 1700
-F 0 "#PWR028" H 2200 1450 50  0001 C CNN
+F 0 "#PWR027" H 2200 1450 50  0001 C CNN
 F 1 "GND" H 2200 1550 50  0000 C CNN
 F 2 "" H 2200 1700 50  0001 C CNN
@@
 $EndComp
 $Comp
-L GND #PWR029
+L GND #PWR028
 U 1 1 5AA01F17
 P 2600 1700
-F 0 "#PWR029" H 2600 1450 50  0001 C CNN
+F 0 "#PWR028" H 2600 1450 50  0001 C CNN
 F 1 "GND" H 2600 1550 50  0000 C CNN
 F 2 "" H 2600 1700 50  0001 C CNN
@@
 $EndComp
 $Comp
-L Jumper_NC_Small JP3
+L Jumper_NO_Small JP3
 U 1 1 5AA02D96
 P 3150 1100
 F 0 "JP3" H 3000 1000 50  0000 C CNN
 F 1 "EXT_EN" H 3250 1000 50  0000 C CNN
-F 2 "TI_conn:JMP" H 3150 1100 50  0001 C CNN
+F 2 "TI_conn:JMP_NO" H 3150 1100 50  0001 C CNN
 F 3 "" H 3150 1100 50  0001 C CNN
 	1    3150 1100
@@
 $EndComp
 $Comp
-L GND #PWR030
+L GND #PWR029
 U 1 1 5AA0500D
 P 3750 3200
-F 0 "#PWR030" H 3750 2950 50  0001 C CNN
+F 0 "#PWR029" H 3750 2950 50  0001 C CNN
 F 1 "GND" H 3750 3050 50  0000 C CNN
 F 2 "" H 3750 3200 50  0001 C CNN
@@
 $EndComp
 $Comp
-L +5V #PWR031
+L +5V #PWR030
 U 1 1 5AA05191
 P 3750 2650
-F 0 "#PWR031" H 3750 2500 50  0001 C CNN
+F 0 "#PWR030" H 3750 2500 50  0001 C CNN
 F 1 "+5V" H 3750 2790 50  0000 C CNN
 F 2 "" H 3750 2650 50  0001 C CNN
@@
 $EndComp
 $Comp
-L GND #PWR032
+L GND #PWR031
 U 1 1 5AA05AC7
 P 6500 3050
-F 0 "#PWR032" H 6500 2800 50  0001 C CNN
+F 0 "#PWR031" H 6500 2800 50  0001 C CNN
 F 1 "GND" H 6500 2900 50  0000 C CNN
 F 2 "" H 6500 3050 50  0001 C CNN
@@
 $EndComp
 $Comp
-L +3.3V #PWR033
+L +3.3V #PWR032
 U 1 1 5AA05AD3
 P 6500 2650
-F 0 "#PWR033" H 6500 2500 50  0001 C CNN
+F 0 "#PWR032" H 6500 2500 50  0001 C CNN
 F 1 "+3.3V" H 6500 2790 50  0000 C CNN
 F 2 "" H 6500 2650 50  0001 C CNN
@@
 EN
 $Comp
-L GND #PWR034
+L GND #PWR033
 U 1 1 5AA0AC76
 P 1650 7400
-F 0 "#PWR034" H 1650 7150 50  0001 C CNN
+F 0 "#PWR033" H 1650 7150 50  0001 C CNN
 F 1 "GND" H 1650 7250 50  0000 C CNN
 F 2 "" H 1650 7400 50  0001 C CNN
@@
 CTL_DRV1
 $Comp
-L GND #PWR035
+L GND #PWR034
 U 1 1 5AA1183B
 P 10250 1700
-F 0 "#PWR035" H 10250 1450 50  0001 C CNN
+F 0 "#PWR034" H 10250 1450 50  0001 C CNN
 F 1 "GND" H 10250 1550 50  0000 C CNN
 F 2 "" H 10250 1700 50  0001 C CNN
@@
 $EndComp
 $Comp
-L +3.3V #PWR036
+L +3.3V #PWR035
 U 1 1 5AA118C9
 P 9700 800
-F 0 "#PWR036" H 9700 650 50  0001 C CNN
+F 0 "#PWR035" H 9700 650 50  0001 C CNN
 F 1 "+3.3V" H 9700 940 50  0000 C CNN
 F 2 "" H 9700 800 50  0001 C CNN
@@
 $EndComp
 $Comp
-L GND #PWR037
+L GND #PWR036
 U 1 1 5AA11B02
 P 8750 1700
-F 0 "#PWR037" H 8750 1450 50  0001 C CNN
+F 0 "#PWR036" H 8750 1450 50  0001 C CNN
 F 1 "GND" H 8750 1550 50  0000 C CNN
 F 2 "" H 8750 1700 50  0001 C CNN
@@
 $EndComp
 $Comp
-L +3.3V #PWR038
+L +3.3V #PWR037
 U 1 1 5AA1515C
 P 8200 800
-F 0 "#PWR038" H 8200 650 50  0001 C CNN
+F 0 "#PWR037" H 8200 650 50  0001 C CNN
 F 1 "+3.3V" H 8200 940 50  0000 C CNN
 F 2 "" H 8200 800 50  0001 C CNN
@@
 $EndComp
 $Comp
-L +3.3V #PWR039
+L +3.3V #PWR038
 U 1 1 5AA17C8F
 P 9950 800
-F 0 "#PWR039" H 9950 650 50  0001 C CNN
+F 0 "#PWR038" H 9950 650 50  0001 C CNN
 F 1 "+3.3V" H 9950 940 50  0000 C CNN
 F 2 "" H 9950 800 50  0001 C CNN
@@
 M_OUT1
 $Comp
-L GND #PWR040
+L GND #PWR039
 U 1 1 5AA1BC55
 P 8200 1700
-F 0 "#PWR040" H 8200 1450 50  0001 C CNN
+F 0 "#PWR039" H 8200 1450 50  0001 C CNN
 F 1 "GND" H 8200 1550 50  0000 C CNN
 F 2 "" H 8200 1700 50  0001 C CNN
@@
 $EndComp
 $Comp
-L GND #PWR041
+L GND #PWR040
 U 1 1 5AA2A5C1
 P 2800 4200
-F 0 "#PWR041" H 2800 3950 50  0001 C CNN
+F 0 "#PWR040" H 2800 3950 50  0001 C CNN
 F 1 "GND" H 2800 4050 50  0000 C CNN
 F 2 "" H 2800 4200 50  0001 C CNN
@@
 $EndComp
 $Comp
-L +3.3V #PWR042
+L +3.3V #PWR041
 U 1 1 5AA2A831
 P 2800 3800
-F 0 "#PWR042" H 2800 3650 50  0001 C CNN
+F 0 "#PWR041" H 2800 3650 50  0001 C CNN
 F 1 "+3.3V" H 2800 3940 50  0000 C CNN
 F 2 "" H 2800 3800 50  0001 C CNN
@@
 $EndComp
 $Comp
-L GND #PWR043
+L GND #PWR042
 U 1 1 5AA2B823
 P 3700 4200
-F 0 "#PWR043" H 3700 3950 50  0001 C CNN
+F 0 "#PWR042" H 3700 3950 50  0001 C CNN
 F 1 "GND" H 3700 4050 50  0000 C CNN
 F 2 "" H 3700 4200 50  0001 C CNN
@@
 $EndComp
 $Comp
-L +3.3V #PWR044
+L +3.3V #PWR043
 U 1 1 5AA2D3AC
 P 9000 4950
-F 0 "#PWR044" H 9000 4800 50  0001 C CNN
+F 0 "#PWR043" H 9000 4800 50  0001 C CNN
 F 1 "+3.3V" H 9000 5090 50  0000 C CNN
 F 2 "" H 9000 4950 50  0001 C CNN
@@
 $EndComp
 $Comp
-L GND #PWR045
+L GND #PWR044
 U 1 1 5AA2DAAB
 P 8900 5500
-F 0 "#PWR045" H 8900 5250 50  0001 C CNN
+F 0 "#PWR044" H 8900 5250 50  0001 C CNN
 F 1 "GND" H 8900 5350 50  0000 C CNN
 F 2 "" H 8900 5500 50  0001 C CNN
@@
 $EndComp
 $Comp
-L +3.3V #PWR046
+L +3.3V #PWR045
 U 1 1 5AA30915
 P 10100 2650
-F 0 "#PWR046" H 10100 2500 50  0001 C CNN
+F 0 "#PWR045" H 10100 2500 50  0001 C CNN
 F 1 "+3.3V" H 10100 2790 50  0000 C CNN
 F 2 "" H 10100 2650 50  0001 C CNN
@@
 $EndComp
 $Comp
-L GND #PWR047
+L GND #PWR046
 U 1 1 5AA3CD30
 P 4550 4200
-F 0 "#PWR047" H 4550 3950 50  0001 C CNN
+F 0 "#PWR046" H 4550 3950 50  0001 C CNN
 F 1 "GND" H 4550 4050 50  0000 C CNN
 F 2 "" H 4550 4200 50  0001 C CNN
@@
 V_IN
 $Comp
-L +5V #PWR048
+L +5V #PWR047
 U 1 1 5AA3EEB8
 P 4800 2650
-F 0 "#PWR048" H 4800 2500 50  0001 C CNN
+F 0 "#PWR047" H 4800 2500 50  0001 C CNN
 F 1 "+5V" H 4800 2790 50  0000 C CNN
 F 2 "" H 4800 2650 50  0001 C CNN
@@
 $EndComp
 $Comp
-L GND #PWR049
+L GND #PWR048
 U 1 1 5AA5712D
 P 5500 3100
-F 0 "#PWR049" H 5500 2850 50  0001 C CNN
+F 0 "#PWR048" H 5500 2850 50  0001 C CNN
 F 1 "GND" H 5500 2950 50  0000 C CNN
 F 2 "" H 5500 3100 50  0001 C CNN
@@
 	8750 1600 8750 1700
 Wire Wire Line
-	8600 900  8600 700
+	8600 700  8600 1300
 Wire Wire Line
 	8600 700  8450 700
@@
 Wire Wire Line
 	8200 1300 8850 1300
-Wire Wire Line
-	8600 1100 8600 1300
 Connection ~ 8600 1300
 Wire Wire Line
@@
 	10050 5600 10050 5700
 Wire Wire Line
-	9650 5450 9650 5600
+	9650 5200 9650 5600
 Connection ~ 9650 5600
 Wire Wire Line
 	9650 4850 9650 5000
-Wire Wire Line
-	9650 5200 9650 5250
 Wire Wire Line
 	2750 4100 2800 4100
@@
 (this is the \nDMA pin)
 $Comp
-L GND #PWR050
+L GND #PWR049
 U 1 1 5AAB0A54
 P 700 1700
-F 0 "#PWR050" H 700 1450 50  0001 C CNN
+F 0 "#PWR049" H 700 1450 50  0001 C CNN
 F 1 "GND" H 700 1550 50  0000 C CNN
 F 2 "" H 700 1700 50  0001 C CNN
@@
 	700  800  700  1100
 $Comp
-L +5V #PWR051
+L +5V #PWR050
 U 1 1 5AAB0BE0
 P 700 800
-F 0 "#PWR051" H 700 650 50  0001 C CNN
+F 0 "#PWR050" H 700 650 50  0001 C CNN
 F 1 "+5V" H 700 940 50  0000 C CNN
 F 2 "" H 700 800 50  0001 C CNN
@@
 Wire Wire Line
 	9650 4850 9950 4850
+Connection ~ 8600 900
+Connection ~ 8600 1100
+Connection ~ 9650 5250
+Connection ~ 9650 5450
 $EndSCHEMATC

Commit message: fixed batt pinout to match h/w v0.0.3 (it's schematic didn't match)
Parts:
- U3: footprint Housings_DFN_QFN:DFN-8-1EP_2x2mm_Pitch0.5mm -> TI_ic:DFN-8-1EP_2x2mm_Pitch0.5mm
Connections:
- net +BATT: now also J1.1 (P1); no longer J1.2 (P2)
- net GND: now also J1.2 (P2); no longer J1.1 (P1)
Changed lines of the file:
@@
 U 1 1 5A9F3996
 P 2550 2900
-F 0 "J1" H 2550 2750 50  0000 C CNN
+F 0 "J1" H 2550 3050 50  0000 C CNN
 F 1 "BATT" V 2650 2900 50  0000 C CNN
 F 2 "Connectors_JST:JST_PH_B2B-PH-K_02x2.00mm_Straight" H 2550 2900 50  0001 C CNN
 F 3 "" H 2550 2900 50  0001 C CNN
 	1    2550 2900
-	-1   0    0    1
+	-1   0    0    -1
 $EndComp
 $Comp
@@
 F 0 "U3" H 8950 1750 50  0000 L CNN
 F 1 "DRV883x" H 9550 1750 50  0000 R CNN
-F 2 "Housings_DFN_QFN:DFN-8-1EP_2x2mm_Pitch0.5mm" H 9250 1050 50  0001 C CNN
+F 2 "TI_ic:DFN-8-1EP_2x2mm_Pitch0.5mm" H 9250 1050 50  0001 C CNN
 F 3 "" H 9250 1450 50  0001 C CNN
 	1    9250 1450

Commit message: nearly finished v1 hardware -- need to finish ground stitching
Parts:
- C4, C5, R1: footprint Capacitors_SMD:C_0805 -> Capacitors_SMD:C_0603
- J2: footprint Connectors_JST:JST_EH_B02B-EH-A_02x2.50mm_Straight -> Connectors_JST:JST_EH_S02B-EH_02x2.50mm_Angled
Changed lines of the file:
@@
 F 0 "J2" H 3450 2750 50  0000 C CNN
 F 1 "5V IN" V 3550 2900 50  0000 C CNN
-F 2 "Connectors_JST:JST_EH_B02B-EH-A_02x2.50mm_Straight" H 3450 2900 50  0001 C CNN
+F 2 "Connectors_JST:JST_EH_S02B-EH_02x2.50mm_Angled" H 3450 2900 50  0001 C CNN
 F 3 "" H 3450 2900 50  0001 C CNN
 	1    3450 2900
@@
 F 0 "C5" H 10260 1570 50  0000 L CNN
 F 1 "0.1uF" H 10260 1420 50  0000 L CNN
-F 2 "Capacitors_SMD:C_0805" H 10250 1500 50  0001 C CNN
+F 2 "Capacitors_SMD:C_0603" H 10250 1500 50  0001 C CNN
 F 3 "" H 10250 1500 50  0001 C CNN
 	1    10250 1500
@@
 F 0 "R1" H 9980 1020 50  0000 L CNN
 F 1 "10k" H 9980 960 50  0000 L CNN
-F 2 "Capacitors_SMD:C_0805" H 9950 1000 50  0001 C CNN
+F 2 "Capacitors_SMD:C_0603" H 9950 1000 50  0001 C CNN
 F 3 "" H 9950 1000 50  0001 C CNN
 	1    9950 1000
@@
 F 0 "C4" H 8210 1570 50  0000 L CNN
 F 1 "0.1uF" H 8210 1420 50  0000 L CNN
-F 2 "Capacitors_SMD:C_0805" H 8200 1500 50  0001 C CNN
+F 2 "Capacitors_SMD:C_0603" H 8200 1500 50  0001 C CNN
 F 3 "" H 8200 1500 50  0001 C CNN
 	1    8200 1500
